File: PCB/Impedance/CC2533_PCB_Main.sch (EAGLE design)
At the start: 48 parts

Commit message: Further updated layout with more rough additions
Parts:
- removed U$37, U$38: DRILL_HOLE, CC2530_PCB_TL:DRILL_HOLE
Connections:
- net RESET: no longer U$37.1, U$38.1
Changed lines of the file:
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@@
 <part name="U$35" library="CC2530_PCB_TL" deviceset="DRILL_HOLE" device=""/>
 <part name="U$36" library="CC2530_PCB_TL" deviceset="DRILL_HOLE" device=""/>
-<part name="U$37" library="CC2530_PCB_TL" deviceset="DRILL_HOLE" device=""/>
-<part name="U$38" library="CC2530_PCB_TL" deviceset="DRILL_HOLE" device=""/>
 <part name="U$39" library="CC2530_PCB_TL" deviceset="X32.768KHZ" device=""/>
 <part name="U$40" library="CC2530_PCB_TL" deviceset="0201" device=""/>
@@
 <instance part="U$35" gate="G$1" x="109.22" y="53.34"/>
 <instance part="U$36" gate="G$1" x="96.52" y="124.46"/>
-<instance part="U$37" gate="G$1" x="81.28" y="124.46"/>
-<instance part="U$38" gate="G$1" x="86.36" y="30.48"/>
 <instance part="U$39" gate="G$1" x="106.68" y="106.68"/>
 <instance part="U$40" gate="G$1" x="124.46" y="119.38"/>
@@
 <pinref part="U$1" gate="G$1" pin="RESET_N"/>
 <wire x1="86.36" y1="33.02" x2="86.36" y2="30.48" width="0.1524" layer="91"/>
-<pinref part="U$38" gate="G$1" pin="1"/>
 </segment>
 <segment>
 <pinref part="U$17" gate="G$1" pin="3"/>
 <wire x1="81.28" y1="127" x2="81.28" y2="124.46" width="0.1524" layer="91"/>
-<pinref part="U$37" gate="G$1" pin="1"/>
 </segment>
 </net>
@@
 <net name="P0_3" class="0">
 <segment>
+<pinref part="U$13" gate="G$1" pin="NC2"/>
+<wire x1="10.16" y1="-12.7" x2="12.7" y2="-12.7" width="0.1524" layer="91"/>
+</segment>
+<segment>
 <pinref part="U$1" gate="G$1" pin="P0_3"/>
 <wire x1="76.2" y1="33.02" x2="76.2" y2="27.94" width="0.1524" layer="91"/>
-</segment>
-<segment>
-<pinref part="U$13" gate="G$1" pin="NC2"/>
-<wire x1="10.16" y1="-12.7" x2="12.7" y2="-12.7" width="0.1524" layer="91"/>
 </segment>
 </net>
@@
 <pinref part="U$29" gate="G$1" pin="2"/>
 <wire x1="-17.78" y1="71.12" x2="-17.78" y2="58.42" width="0.1524" layer="91"/>
-</segment>
-</net>
-<net name="N$35" class="0">
-<segment>
-<pinref part="U$29" gate="G$1" pin="1"/>
-<pinref part="U$1" gate="G$1" pin="P1_5"/>
-<wire x1="10.16" y1="58.42" x2="45.72" y2="58.42" width="0.1524" layer="91"/>
 </segment>
 </net>
@@
 </segment>
 </net>
+<net name="N$24" class="0">
+<segment>
+<pinref part="U$29" gate="G$1" pin="1"/>
+<pinref part="U$1" gate="G$1" pin="P1_5"/>
+<wire x1="10.16" y1="58.42" x2="45.72" y2="58.42" width="0.1524" layer="91"/>
+</segment>
+</net>

Commit message: Update
Parts:
- removed U$34, U$35: DRILL_HOLE, CC2530_PCB_TL:DRILL_HOLE
Connections:
- net VDD: no longer U$34.1, U$35.1
Changed lines of the file:
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@@
 <part name="U$32" library="CC2530_PCB_TL" deviceset="DRILL_HOLE" device=""/>
 <part name="U$33" library="CC2530_PCB_TL" deviceset="DRILL_HOLE" device=""/>
-<part name="U$34" library="CC2530_PCB_TL" deviceset="DRILL_HOLE" device=""/>
-<part name="U$35" library="CC2530_PCB_TL" deviceset="DRILL_HOLE" device=""/>
 <part name="U$36" library="CC2530_PCB_TL" deviceset="DRILL_HOLE" device=""/>
 <part name="U$39" library="CC2530_PCB_TL" deviceset="X32.768KHZ" device=""/>
@@
 <instance part="U$32" gate="G$1" x="198.12" y="58.42"/>
 <instance part="U$33" gate="G$1" x="198.12" y="55.88"/>
-<instance part="U$34" gate="G$1" x="109.22" y="60.96"/>
-<instance part="U$35" gate="G$1" x="109.22" y="53.34"/>
 <instance part="U$36" gate="G$1" x="96.52" y="124.46"/>
 <instance part="U$39" gate="G$1" x="106.68" y="106.68"/>
@@
 <wire x1="109.22" y1="81.28" x2="109.22" y2="66.04" width="0.1524" layer="91"/>
 <wire x1="109.22" y1="66.04" x2="104.14" y2="66.04" width="0.1524" layer="91"/>
-<pinref part="U$34" gate="G$1" pin="1"/>
 <wire x1="109.22" y1="60.96" x2="104.14" y2="60.96" width="0.1524" layer="91"/>
 <pinref part="U$1" gate="G$1" pin="AVDD5"/>
-<wire x1="109.22" y1="53.34" x2="109.22" y2="45.72" width="0.1524" layer="91"/>
 <wire x1="109.22" y1="45.72" x2="104.14" y2="45.72" width="0.1524" layer="91"/>
-<pinref part="U$35" gate="G$1" pin="1"/>
-<pinref part="U$1" gate="G$1" pin="AVDD3"/>
-<wire x1="104.14" y1="53.34" x2="109.22" y2="53.34" width="0.1524" layer="91"/>
 <wire x1="109.22" y1="60.96" x2="109.22" y2="53.34" width="0.1524" layer="91"/>
 <pinref part="U$48" gate="G$1" pin="1"/>
 <junction x="86.36" y="86.36"/>
 <pinref part="U$18" gate="G$1" pin="2"/>
+<wire x1="109.22" y1="53.34" x2="109.22" y2="45.72" width="0.1524" layer="91"/>
 <wire x1="109.22" y1="25.4" x2="109.22" y2="45.72" width="0.1524" layer="91"/>
+<pinref part="U$1" gate="G$1" pin="AVDD3"/>
+<wire x1="104.14" y1="53.34" x2="109.22" y2="53.34" width="0.1524" layer="91"/>
 </segment>
 <segment>
