File: PCB/Impedance/CC2533_PCB_Main.brd (EAGLE design)
At the start: 100 x 40.3 mm, 48 parts

Commit message: Made rough changes to layout traces, updated library with switch outline
Parts:
- moved U$13 27.0 mm to (13.3, 4.70), flipped to the bottom, turned to 0 degrees
- moved U$15 20.0 mm to (13.3, 11.5), flipped to the bottom, turned to 0 degrees
- moved U$20 18.1 mm to (29.4, 24.6)
- moved U$22 14.0 mm to (20.4, 22.1)
- moved U$24 13.4 mm to (12.0, 25.5), turned to 90 degrees
- moved U$23 13.1 mm to (13.8, 23.1)
- moved U$21 12.4 mm to (25.3, 21.5)
- moved U$25 11.9 mm to (13.3, 25.5), turned to 90 degrees
- moved U$26 9.51 mm to (15.8, 25.5), turned to 90 degrees
- moved U$27 8.60 mm to (17.1, 25.5), turned to 90 degrees
- moved U$28 8.00 mm to (18.4, 25.5), turned to 90 degrees
- moved U$19 7.87 mm to (13.2, 17.8), flipped to the bottom
- moved U$16 7.50 mm to (23.7, 16.7)
- moved U$30 4.49 mm to (6.91, 11.7)
- moved U$18 3.32 mm to (50.1, 6.10)
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Connections:
- net N$10: now also U$30.6; no longer U$30.5
- net N$15: now also U$30.2; no longer U$30.1
- net N$30: now also U$30.5; no longer U$30.6
- net N$9: now also U$30.1; no longer U$30.2
Routing:
- net P0_3: track 2.68 -> 47.5 mm, vias 0 -> 1
- net IN1: track 4.65 -> 44.0 mm, vias 0 -> 2
- net RIGHT: track 0.00 -> 32.3 mm, vias 0 -> 1
- net LEFT: track 0.00 -> 30.6 mm, vias 0 -> 3
- net P0_1: track 7.40 -> 35.9 mm, vias 0 -> 1
- net N$31: track 0.00 -> 27.5 mm, vias 0 -> 2
- net VDD: track 33.4 -> 56.8 mm
- net GND: track 26.9 -> 49.9 mm, vias 0 -> 3
- net N$9: track 0.00 -> 19.6 mm, vias 0 -> 1
- net N$32: track 0.00 -> 17.9 mm
- net N$7: track 0.00 -> 13.5 mm
- net N$15: track 0.00 -> 13.4 mm, vias 0 -> 1
- net N$8: track 0.00 -> 11.7 mm
- net N$10: track 0.00 -> 9.60 mm, vias 0 -> 1
- net N$30: track 0.00 -> 5.31 mm, vias 0 -> 1
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Other:
- board size 100 x 40.3 mm -> 69.5 x 40.3 mm

Commit message: Further updated layout with more rough additions
Parts:
- removed U$37, U$38: DRILL_HOLE, CC2530_PCB_TL:DRILL_HOLE
- moved U$24 19.1 mm to (30.0, 19.1), turned to 180 degrees
- moved U$25 17.1 mm to (29.8, 20.9), turned to 270 degrees
- moved U$27 15.8 mm to (31.7, 19.3), turned to 180 degrees
- moved U$28 14.1 mm to (31.6, 20.8), turned to 180 degrees
- moved U$26 8.47 mm to (23.4, 21.8)
- moved U$21 5.63 mm to (20.2, 19.1), turned to 90 degrees
- moved U$13 5.22 mm to (11.2, 9.45)
- moved U$15 5.22 mm to (11.1, 16.3)
- moved U$19 5.22 mm to (11.1, 22.6)
- moved U$30 5.22 mm to (4.75, 16.5)
- moved U$23 4.75 mm to (18.5, 23.6), turned to 270 degrees
- moved U$22 2.56 mm to (18.3, 20.6), turned to 90 degrees
- moved U$20 2.31 mm to (31.6, 23.9)
- moved U$6 1.96 mm to (61.9, 15.2)
- moved U$16 1.88 mm to (25.3, 15.7)
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Connections:
- net RESET: no longer U$37.1, U$38.1
Routing:
- net VDD: track 56.8 -> 105.0 mm, vias 0 -> 4
- net GND: track 49.9 -> 85.9 mm, vias 3 -> 5
- net N$29: track 0.00 -> 32.9 mm, vias 0 -> 1
- net N$25: track 0.00 -> 27.7 mm
- net N$28: track 0.00 -> 20.1 mm
- net N$11: track 0.00 -> 18.4 mm, vias 0 -> 1
- net N$27: track 0.00 -> 13.5 mm
- net RESET: track 1.07 -> 14.0 mm, vias 0 -> 2
- net N$23: track 0.00 -> 10.2 mm
- net RIGHT: track 32.3 -> 42.1 mm
- net N$13: track 0.00 -> 9.39 mm
- net N$14: track 0.00 -> 9.23 mm
- net IN1: track 44.0 -> 52.8 mm
- net N$19: track 0.00 -> 8.01 mm
- net LEFT: track 30.6 -> 37.5 mm
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
Commit message: Update
Parts:
- removed U$34, U$35: DRILL_HOLE, CC2530_PCB_TL:DRILL_HOLE
- moved U$26 5.33 mm to (28.5, 20.3), turned to 270 degrees
- moved U$16 4.88 mm to (30.2, 15.7)
- moved U$31 4.83 mm to (36.8, 19.4), turned to 90 degrees
- moved U$25 2.05 mm to (31.9, 20.8), turned to 0 degrees
- moved U$24 1.97 mm to (31.9, 19.8), turned to 0 degrees
- moved U$27 1.50 mm to (30.2, 19.8), turned to 0 degrees
- moved U$28 1.42 mm to (30.2, 20.8), turned to 0 degrees
- moved U$20 1.42 mm to (30.2, 23.9)
- moved U$29 1.34 mm to (36.7, 17.4), turned to 90 degrees
- moved U$48 0.13 mm to (44.6, 19.4)
- moved U$14 0.13 mm to (38.3, 19.9)
Connections:
- net VDD: no longer U$34.1, U$35.1
Routing:
- net IN2: track 4.65 -> 48.3 mm, vias 0 -> 1
- net VDD: track 105.0 -> 138.3 mm, vias 4 -> 6
- net GND: track 85.9 -> 64.8 mm, vias 5 -> 3
- net N$28: track 20.1 -> 8.12 mm, vias 0 -> 2
- net N$27: track 13.5 -> 7.87 mm
- net N$14: track 9.23 -> 4.32 mm
- net N$6: track 4.12 -> 9.00 mm
- net N$23: track 10.2 -> 15.0 mm
- net N$13: track 9.39 -> 4.65 mm
- net N$19: track 8.01 -> 9.78 mm
- net N$29: track 32.9 -> 31.5 mm
- net N$25: track 27.7 -> 26.3 mm
- net N$11: track 18.4 -> 17.0 mm
- net N$18: track 0.00 -> 0.96 mm
- net RIGHT: track 42.1 -> 41.4 mm
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
Commit message: New changes
Parts:
- moved U$13 30.3 mm to (41.4, 9.11), flipped to the top, turned to 180 degrees
- moved U$15 21.1 mm to (31.0, 9.11), flipped to the top
- moved U$19 17.7 mm to (28.7, 23.4), flipped to the top, turned to 90 degrees
- moved U$23 13.4 mm to (31.9, 23.0)
- moved U$22 9.15 mm to (25.0, 14.4), turned to 270 degrees
- moved U$20 5.46 mm to (35.7, 23.5)
- moved U$21 5.13 mm to (25.0, 17.3), turned to 270 degrees
- moved U$26 4.47 mm to (33.0, 20.3)
- moved U$27 4.06 mm to (34.3, 19.8)
- moved U$28 4.06 mm to (34.3, 20.8)
- moved U$25 4.06 mm to (35.9, 20.8)
- moved U$24 4.05 mm to (35.9, 19.8)
- moved U$16 0.51 mm to (30.7, 15.7)
- moved U$29 0.17 mm to (36.5, 17.4)
Routing:
- net N$9: track 19.6 -> 74.3 mm, vias 1 -> 2
- net P0_3: track 45.3 -> 4.98 mm, vias 1 -> 0
- net VDD: track 138.3 -> 101.2 mm, vias 6 -> 5
- net RIGHT: track 41.4 -> 10.8 mm, vias 1 -> 0
- net N$29: track 31.5 -> 2.12 mm, vias 1 -> 0
- net P0_1: track 33.3 -> 4.04 mm, vias 1 -> 0
- net IN2: track 48.3 -> 24.4 mm, vias 1 -> 0
- net LEFT: track 37.5 -> 16.4 mm, vias 3 -> 0
- net N$31: track 27.5 -> 46.5 mm
- net IN1: track 52.9 -> 33.9 mm, vias 2 -> 0
- net N$15: track 13.4 -> 0.00 mm, vias 1 -> 0
- net N$23: track 15.0 -> 3.83 mm
- net N$10: track 9.60 -> 0.00 mm, vias 1 -> 0
- net N$32: track 17.9 -> 27.5 mm, vias 0 -> 2
- net GND: track 64.8 -> 73.8 mm, vias 3 -> 4
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