File: PCB/Impedance/CC2533_PCB_Biphasic.sch (EAGLE design)
At the start: 40 parts

Commit message: Complete layouts for CC2533 circuits with AD5933
CC2533_PCB_Main_Plane - Voltage stim + Impedance Analysis.
CC2533_PCB_Biphasic - Current stim + Impedance Analysis.
CC2533_PCB_AD5933 - Impedance Analysis only.
Parts:
- removed U$42, U$43, U$48: DRILL_HOLE, CC2530_PCB_TL:DRILL_HOLE
- added U$34: AD8606_OPAMP, CC2530_PCB_TL:AD8606_OPAMP
- added U$35: MP42100, CC2530_PCB_TL:MP42100
- added U$37: NPN_2SC3707, CC2530_PCB_TL:NPN_2SC3707
- added U$38: DRILL_HOLE, CC2530_PCB_TL:DRILL_HOLE
- U$29: value 0603_RES -> DRILL_HOLE; device CC2530_PCB_TL:0603_RES -> CC2530_PCB_TL:DRILL_HOLE
- U$31: value 0402 -> DRILL_HOLE; device CC2530_PCB_TL:0402 -> CC2530_PCB_TL:DRILL_HOLE; RES 1k -> (none)
- U$32, U$33: value DRILL_HOLE -> AS1753_QUAD_SPST; device CC2530_PCB_TL:DRILL_HOLE -> CC2530_PCB_TL:AS1753_QUAD_SPST
- U$36: value DRILL_HOLE -> NPN_2SC3707; device CC2530_PCB_TL:DRILL_HOLE -> CC2530_PCB_TL:NPN_2SC3707
Connections:
- removed net IN1: U$1.P1_1, U$13.IN1, U$13.IN2, U$15.IN1, U$15.IN2
- removed net IN2: U$1.P1_6, U$19.IN1, U$19.IN2
- removed net N$34: U$29.2, U$31.1
- new net B1: U$34.OUTA, U$36.B
- new net B2: U$34.OUTB, U$37.B
- new net C1: U$32.NC2, U$32.NO3, U$36.C
- new net C2: U$33.NC2, U$33.NO3, U$37.C
- new net CLK: U$1.P1_5, U$35.SCK
- new net CS: U$1.P1_1, U$35.CS-BAR
- new net E1: U$34.-INA, U$35.PB1, U$35.PW1, U$36.E
- new net E2: U$34.-INB, U$35.PB0, U$35.PW0, U$37.E
- new net IN_5933: U$1.P2_0, U$19.IN1, U$19.IN2
- new net IN_W: U$1.P1_0, U$13.IN1, U$13.IN2, U$15.IN1, U$15.IN2
- new net I_LEFT: U$15.NC1, U$33.COM1, U$33.COM2
- new net I_LEFT_REF: U$13.NC1, U$33.COM3, U$33.COM4
- new net I_RIGHT: U$15.NC2, U$32.COM1, U$32.COM2
- new net I_RIGHT_REF: U$13.NC2, U$32.COM3, U$32.COM4
- new net MISO: U$1.P1_7, U$32.IN1, U$32.IN2, U$32.IN3, U$32.IN4, U$33.IN1, U$33.IN2, U$33.IN3, U$33.IN4
- new net MOSI: U$1.P1_6, U$35.SI
- net GND: now also U$32.GND, U$33.GND, U$34.V-, U$35.PA0, U$35.PA1, U$35.VSS; no longer U$31.2, U$42.1, U$43.1
- net LEFT: now also U$34.+INB; no longer U$15.NC1
- net N$1: no longer U$32.1
- net N$2: no longer U$33.1
- net N$24: now also U$1.P0_5; no longer U$1.P1_5
- net P0_1: now also U$38.1; no longer U$13.NC1
- net P0_3: now also U$31.1; no longer U$13.NC2
- net RIGHT: now also U$34.+INA; no longer U$15.NC2
- net VDD: now also U$32.NC4, U$32.NO1, U$32.V+, U$33.NC4, U$33.NO1, U$33.V+, U$34.V+, U$35.VDD; no longer U$36.1, U$48.1
